File: capstone_core/capstone_core.kicad_sch (KiCad schematic)
At the start: 6 parts, among them J1 Conn_01x02_Socket, J2 Conn_01x02_Socket, J3 Conn_01x10_Socket, J4 Conn_01x10_Socket, J5 Conn_02x20_Counter_Clockwise, J6 Conn_01x02_Socket

Commit message: adding 10 pin connector footprint
Parts:
- J3, J4: footprint (none) -> Capstone Footprints:CON10_P100X100-RIBBON_TYC
Changed lines of the file:
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@@
 			)
 		)
-		(property "Footprint" ""
+		(property "Footprint" "Capstone Footprints:CON10_P100X100-RIBBON_TYC"
 			(at 154.94 96.52 0)
 			(effects
@@
 			)
 		)
-		(property "Footprint" ""
+		(property "Footprint" "Capstone Footprints:CON10_P100X100-RIBBON_TYC"
 			(at 69.85 95.25 0)
 			(effects
